File: GCU-ADU.kicad_sch (KiCad schematic)
At the start: 5 parts, among them X1 SW_Push, Y1 SW_Push

Commit message: Add switches to schematic
Parts:
- A1, B1, X1, Y1: footprint Button_Switch_SMD:SW_Push_1P1T_NO_6x6mm_H9.5mm -> hhl:SKRR
Changed lines of the file:
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@@
 			)
 		)
-		(property "Footprint" "Button_Switch_SMD:SW_Push_1P1T_NO_6x6mm_H9.5mm"
+		(property "Footprint" "hhl:SKRR"
 			(at 128.27 62.23 0)
 			(effects
@@
 			)
 		)
-		(property "Footprint" "Button_Switch_SMD:SW_Push_1P1T_NO_6x6mm_H9.5mm"
+		(property "Footprint" "hhl:SKRR"
 			(at 128.27 52.07 0)
 			(effects
@@
 			)
 		)
-		(property "Footprint" "Button_Switch_SMD:SW_Push_1P1T_NO_6x6mm_H9.5mm"
+		(property "Footprint" "hhl:SKRR"
 			(at 128.27 41.91 0)
 			(effects
@@
 			)
 		)
-		(property "Footprint" "Button_Switch_SMD:SW_Push_1P1T_NO_6x6mm_H9.5mm"
+		(property "Footprint" "hhl:SKRR"
 			(at 128.27 72.39 0)
 			(effects
